File: Projects/ZMini/ZMini.kicad_pcb (KiCad board)
At the start: 2 copper layers, 127 x 73.7 mm, 58 parts, among them IC1 PO_RESET, IC2 AT28C256B-15PU, IC3 AS6C62256-55PCN, J1 02x20, J2 01x08, J3 01x08, J4 PARENT INT. SEL., J5 USB_OTG, J6 CLOCK DIV., SW1 RESET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

Commit message: added a memory selector and other stuff
Parts:
- added J7: PSW, Pin_Headers:Pin_Header_Straight_1x02_Pitch2.54mm, F.Cu at (210.6, 90.4)
- added R12: 10K, Resistors_THT:R_Axial_DIN0207_L6.3mm_D2.5mm_P10.16mm_Horizontal, F.Cu at (102.0, 121.9)
- added SW2: ONBOARD MEM., Buttons_Switches_THT:SW_DIP_x1_W7.62mm_Slide, F.Cu at (107.4, 121.9)
- J2, J3: footprint Pin_Headers:Pin_Header_Straight_1x08_Pitch2.54mm -> Socket_Strips:Socket_Strip_Straight_1x08_Pitch2.54mm
- moved D3 7.81 mm to (206.9, 103.7)
- moved R11 7.81 mm to (202.5, 103.7)
- moved R4 4.34 mm to (91.8, 109.2)
- moved R5 4.34 mm to (91.8, 112.4)
- moved R3 4.34 mm to (91.8, 115.5)
- moved R6 4.34 mm to (91.8, 118.7)
- moved D2 3.94 mm to (206.9, 97.7)
- moved R10 3.94 mm to (202.5, 97.7)
- moved R7 3.28 mm to (206.1, 114.8), turned to 180 degrees
- moved D1 2.41 mm to (203.8, 111.0)
Connections:
- IC2 pad 20: /A15 -> /ROM_SEL
- J5 pad 1: VCC -> Net-(J5-Pad1)
- U1 pad 1: (no net) -> /A15
- U1 pad 2: (no net) -> /ONB_MEM
- U1 pad 3: (no net) -> /ROM_SEL
- U1 pad 4: (no net) -> Net-(U1-Pad4)
- U1 pad 5: (no net) -> /ONB_MEM
- U1 pad 6: (no net) -> /RAM_SEL
- U2 pad 5: /A15 -> /ROM_SEL
- U2 pad 6: /RAM_SEL -> Net-(U1-Pad4)
Routing:
- net /ROM_SEL: track 0.00 -> 93.7 mm, vias 0 -> 3
- net Net-(U1-Pad4): track 0.00 -> 74.6 mm, vias 0 -> 3
- net /ONB_MEM: track 0.00 -> 55.1 mm, vias 0 -> 2
- net /RAM_SEL: track 78.4 -> 44.4 mm, vias 3 -> 1
- net Net-(D3-Pad1): track 29.2 -> 39.2 mm
- net Net-(J5-Pad1): track 0.00 -> 9.03 mm
- net Net-(D2-Pad1): track 49.3 -> 44.3 mm
- net /~RESET: track 195.0 -> 200.1 mm
- net /~INT: track 127.1 -> 131.7 mm
- net /~NMI: track 100.9 -> 105.6 mm
- net /~WAIT: track 150.0 -> 154.7 mm
- net /~CLK: track 184.8 -> 187.2 mm, vias 3 -> 4
- net /CLK_03: track 47.9 -> 46.3 mm
- net /A15: track 99.3 -> 100.5 mm
- net /CLK_01: track 70.7 -> 71.5 mm, vias 2 -> 3
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Other:
- board text added: "1"
- board text added: "2"
- board text added: "39"
- board text added: "40"
- board text added: "OFF"
- board text added: "ON"
- board text added: "RetroZ SBC"
- board text removed: "ZMini SBC"

Commit message: added the memory board sense
Parts:
- removed G***: LOGO, Libraries:gamma
- removed SW2: ONBOARD MEM., Buttons_Switches_THT:SW_DIP_x1_W7.62mm_Slide
- moved R12 3.76 mm to (105.8, 122.2)
- moved R4 3.76 mm to (95.6, 109.4)
- moved R5 3.76 mm to (95.6, 112.6)
- moved R3 3.76 mm to (95.6, 115.8)
- moved R6 3.76 mm to (95.6, 119.0)
Connections:
- J2 pad 1: GND -> /MEM_EXT
- R12 pad 1: /ONB_MEM -> /MEM_EXT
- R12 pad 2: VCC -> GND
- U1 pad 2: /ONB_MEM -> /MEM_EXT
- U1 pad 5: /ONB_MEM -> /MEM_EXT
Routing:
- net /ONB_MEM: track 55.1 -> 0.00 mm, vias 2 -> 0
- net /MEM_EXT: track 0.00 -> 48.8 mm, vias 0 -> 2
- net /~RESET: track 200.1 -> 196.2 mm
- net /~WAIT: track 154.7 -> 150.8 mm
- net /~NMI: track 105.6 -> 101.7 mm
- net /~INT: track 131.7 -> 128.1 mm
Other:
- board text added: "MEXT"
- board text removed: "GND"
- board text removed: "OFF"
- board text removed: "ON"
